Commit message: Change Gazebo camera plugin.

File: src/wave_rover_description/urdf/wave_rover.urdf (robot description, URDF)
Before this commit: robot wave_rover, 4 links, 3 joints
Links:
- added link camera_link_optical
Joints:
- added joint camera_optical_joint: type fixed, parent camera_link, child camera_link_optical, origin xyz=0 0 0 rpy=-1.5708 0 -1.5708

File: src/wave_rover_description/urdf/wave_rover.urdf.xacro (robot description, xacro)
@@ -12,5 +12,5 @@
     <collision>
       <geometry>
-        <box size="0.3 0.2 0.1"/> <!-- crude collision approximation -->
+        <box size="0.3 0.2 0.1"/>
       </geometry>
     </collision>
@@ -20,9 +20,9 @@
     </inertial>
   </link>
-  <!-- Bracket Stand (support box for bracket + camera) -->
+  <!-- Bracket Stand -->
   <link name="bracket_stand_link">
     <visual>
       <geometry>
-        <box size="0.045 0.11 0.04"/> <!-- 4.5cm x 11cm x 4cm -->
+        <box size="0.045 0.11 0.04"/>
       </geometry>
       <material name="black">
@@ -34,7 +34,7 @@
     <parent link="base_link"/>
     <child link="bracket_stand_link"/>
-    <origin xyz="0.0 0.0042 0.07" rpy="0 0 0"/> <!-- raise box to sit on top of base -->
+    <origin xyz="0.0 0.0042 0.07" rpy="0 0 0"/>
   </joint>
-  <!-- Bracket -->
+  <!-- Camera Bracket -->
   <link name="camera_bracket_link">
     <visual>
@@ -47,5 +47,5 @@
     <parent link="bracket_stand_link"/>
     <child link="camera_bracket_link"/>
-    <origin xyz="0.0 -0.04 0.02" rpy="0 0 0"/> <!-- place bracket on top of box -->
+    <origin xyz="0.0 -0.04 0.02" rpy="0 0 0"/>
   </joint>
   <!-- Camera -->
@@ -63,7 +63,14 @@
     <parent link="camera_bracket_link"/>
     <child link="camera_link"/>
-    <origin xyz="0.0 -0.03 0.02" rpy="0.349 0 0"/> <!-- 20° tilt down -->
+    <origin xyz="0.0 -0.03 0.02" rpy="0.349 0 0"/>
   </joint>
-  <!-- Gazebo diff drive plugin -->
+  <!-- Optical Frame for Camera -->
+  <link name="camera_link_optical"/>
+  <joint name="camera_optical_joint" type="fixed">
+    <parent link="camera_link"/>
+    <child link="camera_link_optical"/>
+    <origin xyz="0 0 0" rpy="-1.5708 0 -1.5708"/>
+  </joint>
+  <!-- Gazebo Plugins -->
   <gazebo>
     <plugin name="diff_drive_controller" filename="libgazebo_ros_diff_drive.so">
@@ -73,10 +80,9 @@
       <left_joint>left_wheel_joint</left_joint>
       <right_joint>right_wheel_joint</right_joint>
-      ...
+      <!-- Add other necessary parameters here -->
     </plugin>
   </gazebo>
-  <!-- Gazebo depth camera plugin -->
   <gazebo reference="camera_link">
-    <sensor name="realsense_sim" type="depth">
+    <sensor name="camera" type="depth">
       <update_rate>30.0</update_rate>
       <camera>
@@ -92,12 +98,14 @@
         </clip>
       </camera>
-      <plugin name="gazebo_ros_depth_camera" filename="libgazebo_ros_depth_camera.so">
+      <plugin name="camera_controller" filename="libgazebo_ros_camera.so">
         <ros>
           <namespace>/camera</namespace>
         </ros>
         <camera_name>camera</camera_name>
-        <image_topic_name>color/image_raw</image_topic_name>
+        <image_topic_name>image_raw</image_topic_name>
         <depth_image_topic_name>depth/image_raw</depth_image_topic_name>
         <info_topic_name>camera_info</info_topic_name>
+        <point_cloud_topic_name>depth/points</point_cloud_topic_name>
+        <frame_name>camera_link_optical</frame_name>
       </plugin>
     </sensor>
