Commit message: Not sure if anything changed but it seems a bit better just has wrong wheel positions.

File: src/wave_rover_description/urdf/rover.urdf.xacro (robot description, xacro)
@@ -39,5 +39,5 @@
     <origin rpy="0 0 0" xyz="0 0 0" />
       <geometry>
-        <mesh filename="package://wave_rover_description/meshes/wave_rover_model.stl" scale="0.001 0.001 0.001"/>
+        <mesh filename="package://wave_rover_description/meshes/rover_body.stl" scale="0.001 0.001 0.001"/>
       </geometry>
       <material name="grey">
@@ -61,5 +61,5 @@
         <box size="0.045 0.11 0.04"/>
       </geometry>
-      <material name="black">
+      <material name="grey">
         <color rgba="0.1 0.1 0.1 1.0"/>
       </material>
